File: motor_controller_2/mc2.kicad_pcb (KiCad board)
At the start: 2 copper layers, 120 x 55 mm, 66 parts, among them P1 Battery, P2 Servo, P3 Uart, P4 Ultrasound, P5 Motor left, P6 Motor right, P7 ISP, P8 RPi 5V, U1 TS1117E33, U10 ts321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

Commit message: mounting holes for servo added
Parts:
- added REF**: 3mm hole, rzfp:3mm_hole, F.Cu at (96.4, 100.0)
- added REF**: 3mm hole, rzfp:3mm_hole, F.Cu at (123.6, 100.0)
Changed lines of the file:
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@@
     (tracks 629)
     (zones 0)
-    (modules 66)
+    (modules 68)
     (nets 64)
   )
@@
       (net 28 "Net-(R40-Pad2)"))
   )
+  (module rzfp:3mm_hole (layer F.Cu)
+    (at 96.4 100)
+    (fp_text reference REF** (at 0 2.54) (layer F.SilkS)
+      (effects (font (size 1 1) (thickness 0.15)))
+    )
+    (fp_text value "3mm hole" (at 0 -2.54) (layer F.Fab)
+      (effects (font (size 1 1) (thickness 0.15)))
+    )
+    (pad 1 thru_hole circle (at 0 0) (size 3.1 3.1) (drill 3.1) (layers *.Cu *.Mask F.SilkS))
+  )
+  (module rzfp:3mm_hole (layer F.Cu)
+    (at 123.6 100)
+    (fp_text reference REF** (at 0 2.54) (layer F.SilkS)
+      (effects (font (size 1 1) (thickness 0.15)))
+    )
+    (fp_text value "3mm hole" (at 0 -2.54) (layer F.Fab)
+      (effects (font (size 1 1) (thickness 0.15)))
+    )
+    (pad 1 thru_hole circle (at 0 0) (size 3.1 3.1) (drill 3.1) (layers *.Cu *.Mask F.SilkS))
+  )
   (gr_line (start 167 84) (end 167 102) (angle 90) (layer Margin) (width 0.2))
   (gr_line (start 162 84) (end 167 84) (angle 90) (layer Margin) (width 0.2))
@@
   (gr_line (start 58 78) (end 58 84) (angle 90) (layer Margin) (width 0.2))
   (gr_line (start 53 84) (end 58 84) (angle 90) (layer Margin) (width 0.2))
-  (gr_line (start 125 102) (end 167 102) (angle 90) (layer Margin) (width 0.2))
-  (gr_line (start 95 95) (end 95 102) (angle 90) (layer Margin) (width 0.2))
-  (gr_line (start 95 95) (end 125 95) (angle 90) (layer Margin) (width 0.2))
-  (gr_line (start 125 95) (end 125 102) (angle 90) (layer Margin) (width 0.2))
+  (gr_line (start 126 102) (end 167 102) (angle 90) (layer Margin) (width 0.2))
+  (gr_line (start 94 95) (end 94 102) (angle 90) (layer Margin) (width 0.2))
+  (gr_line (start 94 95) (end 126 95) (angle 90) (layer Margin) (width 0.2))
+  (gr_line (start 126 95) (end 126 102) (angle 90) (layer Margin) (width 0.2))
   (gr_line (start 53 57) (end 167 57) (angle 90) (layer Margin) (width 0.2))
   (gr_line (start 167 57) (end 167 78) (angle 90) (layer Margin) (width 0.2))
-  (gr_line (start 53 102) (end 95 102) (angle 90) (layer Margin) (width 0.2))
+  (gr_line (start 53 102) (end 94 102) (angle 90) (layer Margin) (width 0.2))
   (gr_line (start 53 57) (end 53 78) (angle 90) (layer Margin) (width 0.2))
   (gr_line (start 50 105) (end 50 50) (angle 90) (layer Edge.Cuts) (width 0.15))
@@
   (segment (start 73.625 95.875) (end 74.875 94.625) (width 0.8) (layer F.Cu) (net 1))
   (segment (start 74.875 94.625) (end 77.19876 92.30124) (width 0.8) (layer F.Cu) (net 1))
-  (segment (start 128.5 61.6) (end 127.15 61.6) (width 0.5) (layer F.Cu) (net 2) (status 400000))
+  (segment (start 128.5 61.6) (end 127.15 61.6) (width 0.5) (layer F.Cu) (net 2))
   (segment (start 125.25 68.5) (end 119.25 74.5) (width 0.5) (layer B.Cu) (net 2))
   (segment (start 125.25 63.5) (end 125.25 68.5) (width 0.5) (layer B.Cu) (net 2))
@@
   (segment (start 145.5 96.5) (end 154 96.5) (width 0.8) (layer F.Cu) (net 5))
   (segment (start 142 93) (end 145.5 96.5) (width 0.8) (layer F.Cu) (net 5))
-  (segment (start 128.25 87.55) (end 125.7 87.55) (width 0.8) (layer F.Cu) (net 5) (status 400000))
+  (segment (start 128.25 87.55) (end 125.7 87.55) (width 0.8) (layer F.Cu) (net 5))
   (segment (start 121.5 91.75) (end 121.5 93) (width 0.8) (layer F.Cu) (net 5))
   (segment (start 125.7 87.55) (end 121.5 91.75) (width 0.8) (layer F.Cu) (net 5))
@@
   (segment (start 144.73 63.105) (end 141.705 63.105) (width 0.4) (layer F.Cu) (net 43))
   (segment (start 141.705 63.105) (end 141.6 63) (width 0.4) (layer F.Cu) (net 43))
-  (zone (net 5) (net_name GNDPWR) (layer B.Cu) (hatch edge 0.508)
-    (connect_pads (clearance 0.508))
-    (min_thickness 0.4)
-    (fill yes (arc_segments 16) (thermal_gap 0.508) (thermal_bridge_width 0.508))
-    (polygon
-      (pts
-        (xy 167 78) (xy 162 78) (xy 162 84) (xy 167 84) (xy 167 102)
-        (xy 125 102) (xy 125 95) (xy 95 95) (xy 95 90.5) (xy 120.75 90.5)
-        (xy 120.75 86.5) (xy 142.5 86.5) (xy 142.5 71.25) (xy 167 71.25) (xy 167 78)
-      )
-    )
-  )
-  (zone (net 5) (net_name GNDPWR) (layer F.Cu) (hatch edge 0.508)
-    (connect_pads (clearance 0.508))
-    (min_thickness 0.4)
-    (fill yes (arc_segments 16) (thermal_gap 0.508) (thermal_bridge_width 0.508))
-    (polygon
-      (pts
-        (xy 167 78) (xy 162 78) (xy 162 84) (xy 167 84) (xy 167 102)
-        (xy 125 102) (xy 125 95) (xy 95 95) (xy 95 90.5) (xy 120.75 90.5)
-        (xy 120.75 86.5) (xy 142.5 86.5) (xy 142.5 71.25) (xy 167 71.25) (xy 167 78)
-      )
-    )
-  )
   (zone (net 2) (net_name GND) (layer F.Cu) (hatch edge 0.508)
     (connect_pads (clearance 0.508))
@@
       )
     )
+  )
+  (zone (net 5) (net_name GNDPWR) (layer B.Cu) (hatch edge 0.508)
+    (connect_pads (clearance 0.508))
+    (min_thickness 0.4)
+    (fill yes (arc_segments 16) (thermal_gap 0.508) (thermal_bridge_width 0.508))
+    (polygon
+      (pts
+        (xy 167 78) (xy 162 78) (xy 162 84) (xy 167 84) (xy 167 102)
+        (xy 126 102) (xy 126 95) (xy 95 95) (xy 95 90.5) (xy 120.75 90.5)
+        (xy 120.75 86.5) (xy 142.5 86.5) (xy 142.5 71.25) (xy 167 71.25) (xy 167 78)
+      )
+    )
+  )
+  (zone (net 5) (net_name GNDPWR) (layer F.Cu) (hatch edge 0.508)
+    (connect_pads (clearance 0.508))
+    (min_thickness 0.4)
+    (fill yes (arc_segments 16) (thermal_gap 0.508) (thermal_bridge_width 0.508))
+    (polygon
+      (pts
+        (xy 167 78) (xy 162 78) (xy 162 84) (xy 167 84) (xy 167 102)
+        (xy 126 102) (xy 126 95) (xy 95 95) (xy 95 90.5) (xy 120.75 90.5)
+        (xy 120.75 86.5) (xy 142.5 86.5) (xy 142.5 71.25) (xy 167 71.25) (xy 167 78)
+      )
+    )

Commit message: pcb design finalized
Parts:
- P4: footprint Pin_Headers:Pin_Header_Straight_1x04 -> Pin_Headers:Pin_Header_Straight_1x06
- moved C63 2.24 mm to (101.2, 73.8), turned to 90 degrees
Connections:
- P4 pad 2: /Pulse_in -> /ADC
- P4 pad 3: /Pulse_out -> /Pulse_in
- P4 pad 4: +3V3 -> /Pulse_out
- P7 pad 3: Net-(P7-Pad3) -> (no net)
- P7 pad 4: Net-(P7-Pad4) -> (no net)
- U6 pad 1: Net-(U6-Pad1) -> (no net)
- U6 pad 11: Net-(U6-Pad11) -> (no net)
- U6 pad 14: Net-(U6-Pad14) -> (no net)
- U6 pad 15: Net-(U6-Pad15) -> (no net)
- U6 pad 16: Net-(U6-Pad16) -> (no net)
- U6 pad 17: Net-(U6-Pad17) -> (no net)
- U6 pad 2: Net-(U6-Pad2) -> (no net)
- U6 pad 24: Net-(U6-Pad24) -> (no net)
- U6 pad 25: Net-(U6-Pad25) -> (no net)
- U6 pad 26: Net-(U6-Pad26) -> (no net)
- U6 pad 27: Net-(U6-Pad27) -> (no net)
- U6 pad 36: Net-(U6-Pad36) -> (no net)
- U6 pad 37: Net-(U6-Pad37) -> (no net)
- U6 pad 40: Net-(U6-Pad40) -> /ADC
- U6 pad 41: Net-(U6-Pad41) -> (no net)
- U6 pad 42: Net-(U6-Pad42) -> (no net)
- U6 pad 43: Net-(U6-Pad43) -> (no net)
- U6 pad 44: Net-(U6-Pad44) -> (no net)
Routing:
- net (no net): track 0.00 -> 700.0 mm
- net /ADC: track 0.00 -> 35.3 mm, vias 0 -> 2
- net +BATT: track 251.7 -> 263.3 mm
- net +5V: track 85.8 -> 96.9 mm
- net +3V3: track 196.8 -> 187.3 mm
- net /Pulse_out: track 12.5 -> 17.1 mm
- net /Pulse_in: track 12.4 -> 14.9 mm
- net GND: track 411.4 -> 413.6 mm
Other:
- board text added: "2.0"
- board text added: "2016 10 18"
- board text added: "Robot Car Motor Control"
- board text added: "Zoltan Raics 2016"
